File: Circuit/power.sch (KiCad schematic (older format))
At the start: 33 parts, among them Q201 FDN340P, Q202 FDN340P, Q203 FDN340P, U201 CN3063, U202 MCP6002

Commit message: First spin at board design.
Parts:
- D6: renamed from D?; footprint (none) -> freetronics_footprints:DIODE_SMA
- R14, R15, R16, R17: renamed from R?; footprint freetronics_footprints:0603 -> Resistors_SMD:R_0603_HandSoldering
- R18, R19: renamed from R?; footprint (none) -> Resistors_SMD:R_0603_HandSoldering
- R201, R202, R204, R205: footprint freetronics_footprints:0603 -> Resistors_SMD:R_0603_HandSoldering
- U201: footprint Plant:CN3063_SOIC8_EP -> libs:CN3063_SOIC8_EP
- U3: renamed from U?; footprint (none) -> TO_SOT_Packages_SMD:SOT-23-6_Handsoldering
- U4: renamed from U?; footprint SOT-23-5 -> TO_SOT_Packages_SMD:SOT-23-5
- gave numbers to parts that had none: 7
Changed lines of the file:
@@
 LIBS:contrib
 LIBS:valves
-LIBS:ESP8266
 LIBS:freetronics_schematic
 LIBS:ESP32-footprints-Shem-Lib
@@
 LIBS:cp2102
 LIBS:ltc3426
-LIBS:InternetOfTux-cache
+LIBS:rotary
+LIBS:IoTuz-cache
 EELAYER 25 0
 EELAYER END
@@
 F 0 "U201" H 3750 3750 60  0000 C CNN
 F 1 "CN3063" H 3800 3650 60  0000 C CNN
-F 2 "Plant:CN3063_SOIC8_EP" H 3900 3550 24  0000 C CNN
+F 2 "libs:CN3063_SOIC8_EP" H 3900 3550 24  0000 C CNN
 F 3 "" H 3800 2900 60  0000 C CNN
 	1    4050 3250
@@
 SOLAR_IN
 $Comp
-L GND #PWR013
+L GND #PWR044
 U 1 1 563C4E24
 P 3950 4650
-F 0 "#PWR013" H 3950 4400 50  0001 C CNN
+F 0 "#PWR044" H 3950 4400 50  0001 C CNN
 F 1 "GND" H 3950 4500 50  0000 C CNN
 F 2 "" H 3950 4650 60  0000 C CNN
@@
 F 0 "R204" V 5030 4150 50  0000 C CNN
 F 1 "7.15K 1%" V 4950 4150 39  0000 C CNN
-F 2 "freetronics_footprints:0603" V 4880 4150 24  0000 C CNN
+F 2 "Resistors_SMD:R_0603_HandSoldering" V 4880 4150 24  0000 C CNN
 F 3 "" H 4950 4150 30  0000 C CNN
 	1    4950 4150
@@
 F 0 "R201" V 1580 1350 50  0000 C CNN
 F 1 "1K" V 1500 1350 50  0000 C CNN
-F 2 "freetronics_footprints:0603" V 1650 1350 24  0000 C CNN
+F 2 "Resistors_SMD:R_0603_HandSoldering" V 1650 1350 24  0000 C CNN
 F 3 "" H 1500 1350 60  0000 C CNN
 	1    1500 1350
@@
 $EndComp
 $Comp
-L GND #PWR014
+L GND #PWR045
 U 1 1 563C5B2C
 P 1150 1500
-F 0 "#PWR014" H 1150 1250 50  0001 C CNN
+F 0 "#PWR045" H 1150 1250 50  0001 C CNN
 F 1 "GND" H 1150 1350 50  0000 C CNN
 F 2 "" H 1150 1500 60  0000 C CNN
@@
 F 0 "R202" V 2600 2650 50  0000 C CNN
 F 1 "1K" V 2700 2650 50  0000 C CNN
-F 2 "freetronics_footprints:0603" V 2800 2650 24  0000 C CNN
+F 2 "Resistors_SMD:R_0603_HandSoldering" V 2800 2650 24  0000 C CNN
 F 3 "" H 2700 2650 60  0000 C CNN
 	1    2700 2650
@@
 Charging current\nIr = 252mA max
 $Comp
-L GND #PWR015
+L GND #PWR046
 U 1 1 56417FB3
 P 7450 4200
-F 0 "#PWR015" H 7450 3950 50  0001 C CNN
+F 0 "#PWR046" H 7450 3950 50  0001 C CNN
 F 1 "GND" H 7450 4050 50  0000 C CNN
 F 2 "" H 7450 4200 60  0000 C CNN
@@
 3.3OUT
 $Comp
-L GND #PWR016
+L GND #PWR047
 U 1 1 5641AA9F
 P 10250 2500
-F 0 "#PWR016" H 10250 2250 50  0001 C CNN
+F 0 "#PWR047" H 10250 2250 50  0001 C CNN
 F 1 "GND" H 10250 2350 50  0000 C CNN
 F 2 "" H 10250 2500 60  0000 C CNN
@@
 $EndComp
 $Comp
-L GND #PWR017
+L GND #PWR048
 U 1 1 5642C1C1
 P 9050 4100
-F 0 "#PWR017" H 9050 3850 50  0001 C CNN
+F 0 "#PWR048" H 9050 3850 50  0001 C CNN
 F 1 "GND" H 9050 3950 50  0000 C CNN
 F 2 "" H 9050 4100 60  0000 C CNN
@@
 $EndComp
 $Comp
-L PWR_FLAG #FLG018
+L PWR_FLAG #FLG049
 U 1 1 5642D1CE
 P 10450 1800
-F 0 "#FLG018" H 10450 1895 50  0001 C CNN
+F 0 "#FLG049" H 10450 1895 50  0001 C CNN
 F 1 "PWR_FLAG" H 10450 1980 50  0000 C CNN
 F 2 "" H 10450 1800 60  0000 C CNN
@@
 $EndComp
 $Comp
-L PWR_FLAG #FLG019
+L PWR_FLAG #FLG050
 U 1 1 5642D5A3
 P 3900 1800
-F 0 "#FLG019" H 3900 1895 50  0001 C CNN
+F 0 "#FLG050" H 3900 1895 50  0001 C CNN
 F 1 "PWR_FLAG" H 3900 1980 50  0000 C CNN
 F 2 "" H 3900 1800 60  0000 C CNN
@@
 $EndComp
 $Comp
-L GND #PWR020
+L GND #PWR051
 U 1 1 5642DA26
 P 10000 4150
-F 0 "#PWR020" H 10000 3900 50  0001 C CNN
+F 0 "#PWR051" H 10000 3900 50  0001 C CNN
 F 1 "GND" H 10000 4000 50  0000 C CNN
 F 2 "" H 10000 4150 60  0000 C CNN
@@
 $EndComp
 $Comp
-L GND #PWR021
+L GND #PWR052
 U 1 1 5642CE9D
 P 4600 2350
-F 0 "#PWR021" H 4600 2100 50  0001 C CNN
+F 0 "#PWR052" H 4600 2100 50  0001 C CNN
 F 1 "GND" H 4600 2200 50  0000 C CNN
 F 2 "" H 4600 2350 60  0000 C CNN
@@
 F 0 "R205" V 5530 3250 50  0000 C CNN
 F 1 "7.15K 1%" V 5450 3250 39  0000 C CNN
-F 2 "freetronics_footprints:0603" V 5350 3250 24  0000 C CNN
+F 2 "Resistors_SMD:R_0603_HandSoldering" V 5350 3250 24  0000 C CNN
 F 3 "" H 5450 3250 60  0000 C CNN
 	1    5450 3250
@@
 	6300 3000 6300 3100
 $Comp
-L GND #PWR022
+L GND #PWR053
 U 1 1 566FA00B
 P 6300 3100
-F 0 "#PWR022" H 6300 2850 50  0001 C CNN
+F 0 "#PWR053" H 6300 2850 50  0001 C CNN
 F 1 "GND" H 6300 2950 50  0000 C CNN
 F 2 "" H 6300 3100 60  0000 C CNN
@@
 	5850 2500 5850 3150
 $Comp
-L R R?
+L R R18
 U 1 1 56EBE55C
 P 6850 3900
-F 0 "R?" V 6930 3900 50  0000 C CNN
+F 0 "R18" V 6930 3900 50  0000 C CNN
 F 1 "100K" V 6850 3900 50  0000 C CNN
-F 2 "" V 6780 3900 50  0000 C CNN
+F 2 "Resistors_SMD:R_0603_HandSoldering" V 6780 3900 50  0001 C CNN
 F 3 "" H 6850 3900 50  0000 C CNN
 	1    6850 3900
@@
 Connection ~ 7450 4100
 $Comp
-L R R?
+L R R19
 U 1 1 56EBECD6
 P 8750 2800
-F 0 "R?" V 8830 2800 50  0000 C CNN
+F 0 "R19" V 8830 2800 50  0000 C CNN
 F 1 "100K" V 8750 2800 50  0000 C CNN
-F 2 "" V 8680 2800 50  0000 C CNN
+F 2 "Resistors_SMD:R_0603_HandSoldering" V 8680 2800 50  0001 C CNN
 F 3 "" H 8750 2800 50  0000 C CNN
 	1    8750 2800
@@
 	6850 3550 7050 3550
 $Comp
-L DIODE_SCHOTTKY D?
+L DIODE_SCHOTTKY D6
 U 1 1 57FA1D94
 P 4150 5950
-F 0 "D?" H 4150 6050 40  0000 C CNN
+F 0 "D6" H 4150 6050 40  0000 C CNN
 F 1 "SS14" H 4150 5850 40  0000 C CNN
-F 2 "" H 4150 5950 60  0000 C CNN
+F 2 "freetronics_footprints:DIODE_SMA" H 4150 5950 60  0001 C CNN
 F 3 "" H 4150 5950 60  0000 C CNN
 	1    4150 5950
@@
 $EndComp
 $Comp
-L INDUCTOR L?
+L INDUCTOR L1
 U 1 1 57FA1E35
 P 3200 5950
-F 0 "L?" V 3150 5950 50  0000 C CNN
+F 0 "L1" V 3150 5950 50  0000 C CNN
 F 1 "2.2uH" V 3300 5950 50  0000 C CNN
-F 2 "" H 3200 5950 50  0000 C CNN
+F 2 "" H 3200 5950 50  0001 C CNN
 F 3 "" H 3200 5950 50  0000 C CNN
 	1    3200 5950
@@
 $EndComp
 $Comp
-L LTC3426 U?
+L LTC3426 U3
 U 1 1 57FA234B
 P 3700 6450
-F 0 "U?" H 3700 5650 60  0000 C CNN
+F 0 "U3" H 3700 5650 60  0000 C CNN
 F 1 "LTC3426" H 3700 7050 60  0000 C CNN
-F 2 "" H 2950 6500 60  0000 C CNN
+F 2 "TO_SOT_Packages_SMD:SOT-23-6_Handsoldering" H 2950 6500 60  0001 C CNN
 F 3 "" H 2950 6500 60  0000 C CNN
 	1    3700 6450
@@
 Connection ~ 3700 5950
 $Comp
-L R R?
+L R R16
 U 1 1 57FA28FE
 P 4600 6200
-F 0 "R?" V 4680 6200 50  0000 C CNN
+F 0 "R16" V 4680 6200 50  0000 C CNN
 F 1 "95.3K" V 4600 6200 39  0000 C CNN
-F 2 "freetronics_footprints:0603" V 4500 6200 24  0001 C CNN
+F 2 "Resistors_SMD:R_0603_HandSoldering" V 4500 6200 24  0001 C CNN
 F 3 "" H 4600 6200 60  0000 C CNN
 	1    4600 6200
@@
 	4600 6350 4600 6650
 $Comp
-L R R?
+L R R17
 U 1 1 57FA322D
 P 4600 6800
-F 0 "R?" V 4680 6800 50  0000 C CNN
+F 0 "R17" V 4680 6800 50  0000 C CNN
 F 1 "30.9K" V 4600 6800 39  0000 C CNN
-F 2 "freetronics_footprints:0603" V 4500 6800 24  0001 C CNN
+F 2 "Resistors_SMD:R_0603_HandSoldering" V 4500 6800 24  0001 C CNN
 F 3 "" H 4600 6800 60  0000 C CNN
 	1    4600 6800
@@
 Connection ~ 4600 6550
 $Comp
-L C C?
+L C C13
 U 1 1 57FA36F6
 P 4850 6550
-F 0 "C?" H 4750 6450 50  0000 L CNN
+F 0 "C13" H 4750 6450 50  0000 L CNN
 F 1 "22uF" H 4650 6650 50  0000 L CNN
 F 2 "freetronics_footprints:1210_CAP" H 5000 6750 24  0001 C CNN
@@
 Connection ~ 4600 7100
 $Comp
-L GND #PWR?
+L GND #PWR054
 U 1 1 57FA4959
 P 4900 7150
-F 0 "#PWR?" H 4900 6900 50  0001 C CNN
+F 0 "#PWR054" H 4900 6900 50  0001 C CNN
 F 1 "GND" H 4900 7000 50  0000 C CNN
 F 2 "" H 4900 7150 50  0000 C CNN
@@
 Connection ~ 4850 7100
 $Comp
-L R R?
+L R R15
 U 1 1 57FA4BF9
 P 3050 6550
-F 0 "R?" V 3130 6550 50  0000 C CNN
+F 0 "R15" V 3130 6550 50  0000 C CNN
 F 1 "1M" V 3050 6550 39  0000 C CNN
-F 2 "freetronics_footprints:0603" V 2950 6550 24  0001 C CNN
+F 2 "Resistors_SMD:R_0603_HandSoldering" V 2950 6550 24  0001 C CNN
 F 3 "" H 3050 6550 60  0000 C CNN
 	1    3050 6550
@@
 Connection ~ 2800 6400
 $Comp
-L C C?
+L C C12
 U 1 1 57FA4E9F
 P 2800 6850
-F 0 "C?" H 2700 6750 50  0000 L CNN
+F 0 "C12" H 2700 6750 50  0000 L CNN
 F 1 "10uF" H 2600 6950 50  0000 L CNN
 F 2 "freetronics_footprints:1210_CAP" H 2950 7050 24  0001 C CNN
@@
 USB_IN
 $Comp
-L DIODE_SCHOTTKY D?
+L DIODE_SCHOTTKY D5
 U 1 1 57FA9576
 P 2150 5300
-F 0 "D?" H 2150 5400 40  0000 C CNN
+F 0 "D5" H 2150 5400 40  0000 C CNN
 F 1 "SS14" H 2150 5200 40  0000 C CNN
 F 2 "freetronics_footprints:DIODE_SMA" H 2150 5150 24  0000 C CNN
@@
 $EndComp
 $Comp
-L MOSFET_P Q?
+L MOSFET_P Q4
 U 1 1 57FA9A8C
 P 1800 5850
-F 0 "Q?" V 1700 5700 60  0000 R CNN
+F 0 "Q4" V 1700 5700 60  0000 R CNN
 F 1 "FDN340P" V 2100 6050 60  0000 R CNN
 F 2 "freetronics_footprints:SOT23_FET" V 2150 5850 24  0000 C CNN
@@
 $EndComp
 $Comp
-L R R?
+L R R14
 U 1 1 57FA9A92
 P 1450 5500
-F 0 "R?" V 1530 5500 50  0000 C CNN
+F 0 "R14" V 1530 5500 50  0000 C CNN
 F 1 "1K" V 1450 5500 50  0000 C CNN
-F 2 "freetronics_footprints:0603" V 1600 5500 24  0000 C CNN
+F 2 "Resistors_SMD:R_0603_HandSoldering" V 1600 5500 24  0000 C CNN
 F 3 "" H 1450 5500 60  0000 C CNN
 	1    1450 5500
@@
 $EndComp
 $Comp
-L GND #PWR?
+L GND #PWR055
 U 1 1 57FA9A98
 P 1150 5650
-F 0 "#PWR?" H 1150 5400 50  0001 C CNN
+F 0 "#PWR055" H 1150 5400 50  0001 C CNN
 F 1 "GND" H 1150 5500 50  0000 C CNN
 F 2 "" H 1150 5650 60  0000 C CNN
@@
 5V_SWITCH
 $Comp
-L Switch_DPST SW?
+L Switch_DPST SW6
 U 1 1 57FB1109
 P 1150 4250
-F 0 "SW?" H 1450 4300 50  0000 C CNN
+F 0 "SW6" H 1450 4300 50  0000 C CNN
 F 1 "POWER" H 1450 4200 50  0000 C CNN
-F 2 "" H 1150 4250 50  0000 C CNN
+F 2 "" H 1150 4250 50  0001 C CNN
 F 3 "" H 1150 4250 50  0000 C CNN
 	1    1150 4250
@@
 5V
 $Comp
-L LD3985M U?
+L LD3985M U4
 U 1 1 57FB1BEE
 P 8750 5600
-F 0 "U?" H 9000 5350 50  0000 C CNN
+F 0 "U4" H 9000 5350 50  0000 C CNN
 F 1 "LD3985M" H 8750 5800 50  0000 C CNN
-F 2 "SOT-23-5" H 8650 5350 50  0000 C CNN
+F 2 "TO_SOT_Packages_SMD:SOT-23-5" H 8650 5350 50  0000 C CNN
 F 3 "" H 8750 5600 50  0000 C CNN
 	1    8750 5600
@@
 3.3V_SWITCH
 $Comp
-L C C?
+L C C14
 U 1 1 57FB2358
 P 9350 5900
-F 0 "C?" H 9250 5800 50  0000 L CNN
+F 0 "C14" H 9250 5800 50  0000 L CNN
 F 1 "100nF" H 9150 6000 50  0000 L CNN
 F 2 "freetronics_footprints:1210_CAP" H 9500 6100 24  0001 C CNN
@@
 	9250 5550 9400 5550
 $Comp
-L GND #PWR?
+L GND #PWR056
 U 1 1 57FB3009
 P 8750 6150
-F 0 "#PWR?" H 8750 5900 50  0001 C CNN
+F 0 "#PWR056" H 8750 5900 50  0001 C CNN
 F 1 "GND" H 8750 6000 50  0000 C CNN
 F 2 "" H 8750 6150 50  0000 C CNN

Commit message: Removed 5V components.
And solar.  At this point they aren't needed.
Parts:
- removed C12: 10uF, freetronics_footprints:1210_CAP, symbol C
- removed C13: 22uF, freetronics_footprints:1210_CAP, symbol C
- removed D5, D6: SS14, freetronics_footprints:DIODE_SMA, symbol DIODE_SCHOTTKY
- removed L1: 2.2uH, symbol INDUCTOR
- removed Q201, Q4: FDN340P, freetronics_footprints:SOT23_FET, symbol MOSFET_P
- removed R14, R201: 1K, Resistors_SMD:R_0603_HandSoldering, symbol R
- removed R15: 1M, Resistors_SMD:R_0603_HandSoldering, symbol R
- removed R16: 95.3K, Resistors_SMD:R_0603_HandSoldering, symbol R
- removed R17: 30.9K, Resistors_SMD:R_0603_HandSoldering, symbol R
- removed SW6: POWER, symbol Switch_DPST
- removed U3: LTC3426, TO_SOT_Packages_SMD:SOT-23-6_Handsoldering, symbol LTC3426
- added SW?: ON/OFF, symbol SPST
- LED201, LED202: footprint freetronics_footprints:LED-0805 -> LEDs:LED_0805
Connections:
- net labels removed: 5OUT, 5V, 5V_SWITCH, SOLAR_IN
- wire segments 99 -> 86
Other:
- note removed: "-Take our 3.3v from our battery\nand produce 5v.\n-If we have 5v from usb,\nignore the battery (circuit is 5v safe)"
- note removed: "SPDT Switch to\nTurn on and OFF"
- note removed: "Solar input:\n7V open circuit voltage panel\nNominal 4-6V under load"
- moved on the sheet: D201
