File: Circuit/IRTransceiver.sch (KiCad schematic (older format))
At the start: 4 parts, among them P8 IRReceiver, Q4 S8050

Commit message: More component information.
Parts:
- removed Q4: S8050, TO_SOT_Packages_SMD:SOT-23_Handsoldering, symbol S8050
- added Q?: MOSFET_N, freetronics_footprints:SOT23_FET, symbol MOSFET_N
- R16: Digikey PN (none) -> 311-22GRCT-ND; Link (none) -> http://www.digikey.com.au/product-detail/en/yageo/RC0603JR-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; Manufacturer PN (none) -> RC0603JR-0722RL; Unit Cost (none) -> 0.10
Connections:
- net +3V3: now also Q?.D
- net IRTx: now also Q?.G
- net at R16.1: now also Q?.S
Other:
- note removed: "Lazy, but we don't have any N-MOS on the design\nand will work just fine."
Changed lines of the file:
@@
 F 2 "Resistors_SMD:R_0603_HandSoldering" V 4430 4150 50  0001 C CNN
 F 3 "" H 4500 4150 50  0000 C CNN
+F 4 "311-22GRCT-ND" V 4500 4150 60  0001 C CNN "Digikey PN"
+F 5 "http://www.digikey.com.au/product-detail/en/yageo/RC0603JR-0722RL/311-22GRCT-ND/729690" V 4500 4150 60  0001 C CNN "Link"
+F 6 "RC0603JR-0722RL" V 4500 4150 60  0001 C CNN "Manufacturer PN"
+F 7 "0.10" V 4500 4150 60  0001 C CNN "Unit Cost"
 	1    4500 4150
 	1    0    0    -1
@@
 Text Notes 4700 4600 0    60   ~ 0
 I_f roughly 90mA @ 1.3V
-Text Notes 4750 3600 0    60   ~ 0
-Lazy, but we don't have any N-MOS on the design\nand will work just fine.
 $Comp
-L S8050 Q4
-U 1 1 581E1075
+L MOSFET_N Q?
+U 1 1 58209DEB
 P 4400 3650
-F 0 "Q4" H 4600 3725 50  0000 L CNN
-F 1 "S8050" H 4600 3650 50  0000 L CNN
-F 2 "TO_SOT_Packages_SMD:SOT-23_Handsoldering" H 4600 3575 50  0000 L CIN
-F 3 "" H 4400 3650 50  0000 L CNN
+F 0 "Q?" H 4310 3820 60  0000 R CNN
+F 1 "MOSFET_N" H 4460 3400 60  0000 R CNN
+F 2 "freetronics_footprints:SOT23_FET" H 4400 3650 60  0000 C CNN
+F 3 "" H 4400 3650 60  0000 C CNN
+F 4 "568-5818-1-ND" H 4400 3650 60  0001 C CNN "Digikey PN"
+F 5 "http://www.digikey.com.au/product-detail/en/nxp-semiconductors/2N7002P,215/568-5818-1-ND/2531105" H 4400 3650 60  0001 C CNN "Link"
+F 6 "2N7002P,215" H 4400 3650 60  0001 C CNN "Manufacturer PN"
+F 7 "0.14" H 4400 3650 60  0001 C CNN "Unit Cost"
 	1    4400 3650
 	1    0    0    -1

Commit message: Updated Alligator tabs
Incomplete.  Included to provide ideas.
Parts:
- gave numbers to parts that had none: 1
Changed lines of the file:
@@
 $EndComp
 $Comp
-L +3.3V #PWR066
+L +3.3V #PWR068
 U 1 1 581D5F60
 P 4050 2750
-F 0 "#PWR066" H 4050 2600 50  0001 C CNN
+F 0 "#PWR068" H 4050 2600 50  0001 C CNN
 F 1 "+3.3V" H 4050 2890 50  0000 C CNN
 F 2 "" H 4050 2750 50  0000 C CNN
@@
 $EndComp
 $Comp
-L GND #PWR067
+L GND #PWR069
 U 1 1 581D5F76
 P 4250 2750
-F 0 "#PWR067" H 4250 2500 50  0001 C CNN
+F 0 "#PWR069" H 4250 2500 50  0001 C CNN
 F 1 "GND" H 4250 2600 50  0000 C CNN
 F 2 "" H 4250 2750 50  0000 C CNN
@@
 	4500 3850 4500 4000
 $Comp
-L GND #PWR068
+L GND #PWR070
 U 1 1 581D6BBC
 P 4500 4950
-F 0 "#PWR068" H 4500 4700 50  0001 C CNN
+F 0 "#PWR070" H 4500 4700 50  0001 C CNN
 F 1 "GND" H 4500 4800 50  0000 C CNN
 F 2 "" H 4500 4950 50  0000 C CNN
@@
 	4050 2950 4050 2750
 $Comp
-L +3.3V #PWR069
+L +3.3V #PWR071
 U 1 1 581D6BFC
 P 4500 3300
-F 0 "#PWR069" H 4500 3150 50  0001 C CNN
+F 0 "#PWR071" H 4500 3150 50  0001 C CNN
 F 1 "+3.3V" H 4500 3440 50  0000 C CNN
 F 2 "" H 4500 3300 50  0000 C CNN
@@
 I_f roughly 90mA @ 1.3V
 $Comp
-L MOSFET_N Q?
+L MOSFET_N Q4
 U 1 1 58209DEB
 P 4400 3650
-F 0 "Q?" H 4310 3820 60  0000 R CNN
+F 0 "Q4" H 4310 3820 60  0000 R CNN
 F 1 "MOSFET_N" H 4460 3400 60  0000 R CNN
 F 2 "freetronics_footprints:SOT23_FET" H 4400 3650 60  0000 C CNN

Commit message: BOM information to schematic. Power & main sheets mostly.
Parts:
- renumbered Q4 to Q?
Changed lines of the file:
@@
 $EndComp
 $Comp
-L +3.3V #PWR068
+L +3.3V #PWR066
 U 1 1 581D5F60
 P 4050 2750
-F 0 "#PWR068" H 4050 2600 50  0001 C CNN
+F 0 "#PWR066" H 4050 2600 50  0001 C CNN
 F 1 "+3.3V" H 4050 2890 50  0000 C CNN
 F 2 "" H 4050 2750 50  0000 C CNN
@@
 $EndComp
 $Comp
-L GND #PWR069
+L GND #PWR067
 U 1 1 581D5F76
 P 4250 2750
-F 0 "#PWR069" H 4250 2500 50  0001 C CNN
+F 0 "#PWR067" H 4250 2500 50  0001 C CNN
 F 1 "GND" H 4250 2600 50  0000 C CNN
 F 2 "" H 4250 2750 50  0000 C CNN
@@
 	4500 3850 4500 4000
 $Comp
-L GND #PWR070
+L GND #PWR068
 U 1 1 581D6BBC
 P 4500 4950
-F 0 "#PWR070" H 4500 4700 50  0001 C CNN
+F 0 "#PWR068" H 4500 4700 50  0001 C CNN
 F 1 "GND" H 4500 4800 50  0000 C CNN
 F 2 "" H 4500 4950 50  0000 C CNN
@@
 	4050 2950 4050 2750
 $Comp
-L +3.3V #PWR071
+L +3.3V #PWR069
 U 1 1 581D6BFC
 P 4500 3300
-F 0 "#PWR071" H 4500 3150 50  0001 C CNN
+F 0 "#PWR069" H 4500 3150 50  0001 C CNN
 F 1 "+3.3V" H 4500 3440 50  0000 C CNN
 F 2 "" H 4500 3300 50  0000 C CNN
@@
 I_f roughly 90mA @ 1.3V
 $Comp
-L MOSFET_N Q4
+L MOSFET_N Q?
 U 1 1 58209DEB
 P 4400 3650
-F 0 "Q4" H 4310 3820 60  0000 R CNN
+F 0 "Q?" H 4310 3820 60  0000 R CNN
 F 1 "MOSFET_N" H 4460 3400 60  0000 R CNN
 F 2 "freetronics_footprints:SOT23_FET" H 4400 3650 60  0000 C CNN

Commit message: Updated alligator clips.
Some basic placement
Parts:
- gave numbers to parts that had none: 1
Changed lines of the file:
@@
 $EndComp
 $Comp
-L +3.3V #PWR066
+L +3.3V #PWR065
 U 1 1 581D5F60
 P 4050 2750
-F 0 "#PWR066" H 4050 2600 50  0001 C CNN
+F 0 "#PWR065" H 4050 2600 50  0001 C CNN
 F 1 "+3.3V" H 4050 2890 50  0000 C CNN
 F 2 "" H 4050 2750 50  0000 C CNN
@@
 $EndComp
 $Comp
-L GND #PWR067
+L GND #PWR066
 U 1 1 581D5F76
 P 4250 2750
-F 0 "#PWR067" H 4250 2500 50  0001 C CNN
+F 0 "#PWR066" H 4250 2500 50  0001 C CNN
 F 1 "GND" H 4250 2600 50  0000 C CNN
 F 2 "" H 4250 2750 50  0000 C CNN
@@
 	4500 3850 4500 4000
 $Comp
-L GND #PWR068
+L GND #PWR067
 U 1 1 581D6BBC
 P 4500 4950
-F 0 "#PWR068" H 4500 4700 50  0001 C CNN
+F 0 "#PWR067" H 4500 4700 50  0001 C CNN
 F 1 "GND" H 4500 4800 50  0000 C CNN
 F 2 "" H 4500 4950 50  0000 C CNN
@@
 	4050 2950 4050 2750
 $Comp
-L +3.3V #PWR069
+L +3.3V #PWR068
 U 1 1 581D6BFC
 P 4500 3300
-F 0 "#PWR069" H 4500 3150 50  0001 C CNN
+F 0 "#PWR068" H 4500 3150 50  0001 C CNN
 F 1 "+3.3V" H 4500 3440 50  0000 C CNN
 F 2 "" H 4500 3300 50  0000 C CNN
@@
 I_f roughly 90mA @ 1.3V
 $Comp
-L MOSFET_N Q?
+L MOSFET_N Q4
 U 1 1 58209DEB
 P 4400 3650
-F 0 "Q?" H 4310 3820 60  0000 R CNN
+F 0 "Q4" H 4310 3820 60  0000 R CNN
 F 1 "MOSFET_N" H 4460 3400 60  0000 R CNN
 F 2 "freetronics_footprints:SOT23_FET" H 4400 3650 60  0000 C CNN
