File: Circuit/IRTransceiver.sch (KiCad schematic (older format))
At the start: 4 parts, among them P8 IRReceiver, Q4 MOSFET_N

Commit message: Some recommendations from Angus.
Parts:
- removed Q4: MOSFET_N, freetronics_footprints:SOT23_FET, symbol MOSFET_N
- added Q4: FDN340P, freetronics_footprints:SOT23_FET, symbol MOSFET_P
- added R?: 10K, Resistors_SMD:R_0603_HandSoldering, symbol R
Connections:
- net +3V3: now also Q4.S, R?.1
- net at R16.1: now also Q4.D
- new net ~IRTx: Q4.G, R?.2
Other:
- moved on the sheet: D3, R16
Changed lines of the file:
@@
 Text Notes 3850 2350 0    60   ~ 0
 38kHz sensitivity. \nSpectrum Cf around 940-950nm.
-Text HLabel 4050 2500 0    60   Output ~ 0
+Text HLabel 3900 2500 0    60   Output ~ 0
 IRRx
 Wire Wire Line
@@
 	4400 2600 4400 2500
 Wire Wire Line
-	4400 2500 4050 2500
+	4400 2500 3900 2500
 $Comp
 L LED D3
 U 1 1 581D68B3
-P 4500 4600
-F 0 "D3" H 4500 4700 50  0000 C CNN
-F 1 "IRLED" H 4500 4500 50  0000 C CNN
-F 2 "LEDs:LED-5MM" H 4500 4600 50  0001 C CNN
-F 3 "" H 4500 4600 50  0000 C CNN
-F 4 "TSAL6200" H 4500 4600 60  0001 C CNN "Manufacturer PN"
-F 5 "751-1204-ND" H 4500 4600 60  0001 C CNN "Digikey PN"
-F 6 "http://www.digikey.com.au/product-detail/en/vishay-semiconductor-opto-division/TSAL6200/751-1204-ND/1681339" H 4500 4600 60  0001 C CNN "Link"
-F 7 "0.57" H 4500 4600 60  0001 C CNN "Unit Cost"
-	1    4500 4600
+P 4500 4800
+F 0 "D3" H 4500 4900 50  0000 C CNN
+F 1 "IRLED" H 4500 4700 50  0000 C CNN
+F 2 "LEDs:LED-5MM" H 4500 4800 50  0001 C CNN
+F 3 "" H 4500 4800 50  0000 C CNN
+F 4 "TSAL6200" H 4500 4800 60  0001 C CNN "Manufacturer PN"
+F 5 "751-1204-ND" H 4500 4800 60  0001 C CNN "Digikey PN"
+F 6 "http://www.digikey.com.au/product-detail/en/vishay-semiconductor-opto-division/TSAL6200/751-1204-ND/1681339" H 4500 4800 60  0001 C CNN "Link"
+F 7 "0.57" H 4500 4800 60  0001 C CNN "Unit Cost"
+	1    4500 4800
 	0    -1   -1   0
 $EndComp
@@
 L R R16
 U 1 1 581D690A
-P 4500 4150
-F 0 "R16" V 4580 4150 50  0000 C CNN
-F 1 "22R" V 4500 4150 50  0000 C CNN
-F 2 "Resistors_SMD:R_0603_HandSoldering" V 4430 4150 50  0001 C CNN
-F 3 "" H 4500 4150 50  0000 C CNN
-F 4 "311-22GRCT-ND" V 4500 4150 60  0001 C CNN "Digikey PN"
-F 5 "http://www.digikey.com.au/product-detail/en/yageo/RC0603JR-0722RL/311-22GRCT-ND/729690" V 4500 4150 60  0001 C CNN "Link"
-F 6 "RC0603JR-0722RL" V 4500 4150 60  0001 C CNN "Manufacturer PN"
-F 7 "0.10" V 4500 4150 60  0001 C CNN "Unit Cost"
-	1    4500 4150
+P 4500 4400
+F 0 "R16" V 4580 4400 50  0000 C CNN
+F 1 "22R" V 4500 4400 50  0000 C CNN
+F 2 "Resistors_SMD:R_0603_HandSoldering" V 4430 4400 50  0001 C CNN
+F 3 "" H 4500 4400 50  0000 C CNN
+F 4 "311-22GRCT-ND" V 4500 4400 60  0001 C CNN "Digikey PN"
+F 5 "http://www.digikey.com.au/product-detail/en/yageo/RC0603JR-0722RL/311-22GRCT-ND/729690" V 4500 4400 60  0001 C CNN "Link"
+F 6 "RC0603JR-0722RL" V 4500 4400 60  0001 C CNN "Manufacturer PN"
+F 7 "0.10" V 4500 4400 60  0001 C CNN "Unit Cost"
+	1    4500 4400
 	1    0    0    -1
 $EndComp
 Wire Wire Line
-	4500 4300 4500 4400
+	4500 4550 4500 4600
 Wire Wire Line
-	4500 3850 4500 4000
+	4500 4150 4500 4250
 $Comp
 L GND #PWR067
 U 1 1 581D6BBC
-P 4500 4950
-F 0 "#PWR067" H 4500 4700 50  0001 C CNN
-F 1 "GND" H 4500 4800 50  0000 C CNN
-F 2 "" H 4500 4950 50  0000 C CNN
-F 3 "" H 4500 4950 50  0000 C CNN
-	1    4500 4950
+P 4500 5100
+F 0 "#PWR067" H 4500 4850 50  0001 C CNN
+F 1 "GND" H 4500 4950 50  0000 C CNN
+F 2 "" H 4500 5100 50  0000 C CNN
+F 3 "" H 4500 5100 50  0000 C CNN
+	1    4500 5100
 	1    0    0    -1
 $EndComp
 Wire Wire Line
-	4500 4800 4500 4950
+	4500 5000 4500 5100
 Wire Wire Line
 	4050 2950 4050 2750
@@
 L +3.3V #PWR068
 U 1 1 581D6BFC
-P 4500 3300
-F 0 "#PWR068" H 4500 3150 50  0001 C CNN
-F 1 "+3.3V" H 4500 3440 50  0000 C CNN
-F 2 "" H 4500 3300 50  0000 C CNN
-F 3 "" H 4500 3300 50  0000 C CNN
-	1    4500 3300
+P 4500 3400
+F 0 "#PWR068" H 4500 3250 50  0001 C CNN
+F 1 "+3.3V" H 4500 3540 50  0000 C CNN
+F 2 "" H 4500 3400 50  0000 C CNN
+F 3 "" H 4500 3400 50  0000 C CNN
+	1    4500 3400
+	1    0    0    -1
+$EndComp
+Text HLabel 3900 3950 0    60   Input ~ 0
+~IRTx
+Text Notes 4700 5000 0    60   ~ 0
+I_f roughly 90mA @ 1.3V
+$Comp
+L MOSFET_P Q4
+U 1 1 582AD6C8
+P 4400 3950
+F 0 "Q4" V 4200 3800 60  0000 R CNN
+F 1 "FDN340P" V 4300 3800 60  0000 R CNN
+F 2 "freetronics_footprints:SOT23_FET" V 4100 3650 24  0000 C CNN
+F 3 "" H 4400 3950 60  0000 C CNN
+F 4 "FDN340PCT-ND" V 4400 3950 60  0001 C CNN "Digikey PN"
+F 5 "http://www.digikey.com.au/product-detail/en/fairchild-semiconductor/FDN340P/FDN340PCT-ND/965604" V 4400 3950 60  0001 C CNN "Link"
+F 6 "FDN340P" V 4400 3950 60  0001 C CNN "Manufacturer PN"
+F 7 "0.39" V 4400 3950 60  0001 C CNN "Unit Cost"
+	1    4400 3950
+	1    0    0    1
+$EndComp
+Wire Wire Line
+	3900 3950 4050 3950
+Wire Wire Line
+	4050 3950 4200 3950
+Wire Wire Line
+	4500 3400 4500 3500
+Wire Wire Line
+	4500 3500 4500 3750
+$Comp
+L R R?
+U 1 1 582B0DCC
+P 4050 3750
+F 0 "R?" V 4130 3750 50  0000 C CNN
+F 1 "10K" V 3950 3750 50  0000 C CNN
+F 2 "Resistors_SMD:R_0603_HandSoldering" V 3980 3750 50  0001 C CNN
+F 3 "" H 4050 3750 50  0000 C CNN
+F 4 "311-10KGRCT-ND" V 4050 3750 60  0001 C CNN "Digikey PN"
+F 5 "http://www.digikey.com.au/product-detail/en/yageo/RC0603JR-0710KL/311-10KGRCT-ND/729647" V 4050 3750 60  0001 C CNN "Link"
+F 6 "RC0603JR-0710KL" V 4050 3750 60  0001 C CNN "Manufacturer PN"
+F 7 "0.10" V 4050 3750 60  0001 C CNN "Unit Cost"
+	1    4050 3750
 	1    0    0    -1
 $EndComp
 Wire Wire Line
-	4500 3300 4500 3450
-Text HLabel 4050 3650 0    60   Input ~ 0
-IRTx
+	4500 3500 4050 3500
 Wire Wire Line
-	4050 3650 4200 3650
-Text Notes 4700 4600 0    60   ~ 0
-I_f roughly 90mA @ 1.3V
-$Comp
-L MOSFET_N Q4
-U 1 1 58209DEB
-P 4400 3650
-F 0 "Q4" H 4310 3820 60  0000 R CNN
-F 1 "MOSFET_N" H 4460 3400 60  0000 R CNN
-F 2 "freetronics_footprints:SOT23_FET" H 4400 3650 60  0000 C CNN
-F 3 "" H 4400 3650 60  0000 C CNN
-F 4 "568-5818-1-ND" H 4400 3650 60  0001 C CNN "Digikey PN"
-F 5 "http://www.digikey.com.au/product-detail/en/nxp-semiconductors/2N7002P,215/568-5818-1-ND/2531105" H 4400 3650 60  0001 C CNN "Link"
-F 6 "2N7002P,215" H 4400 3650 60  0001 C CNN "Manufacturer PN"
-F 7 "0.14" H 4400 3650 60  0001 C CNN "Unit Cost"
-	1    4400 3650
-	1    0    0    -1
-$EndComp
+	4050 3500 4050 3600
+Connection ~ 4500 3500
+Wire Wire Line
+	4050 3900 4050 3950
+Connection ~ 4050 3950
 $EndSCHEMATC

Commit message: More sectioning. Nearly there.
Parts:
- gave numbers to parts that had none: 1
Changed lines of the file:
@@
 $EndComp
 $Comp
-L +3.3V #PWR065
+L +3.3V #PWR067
 U 1 1 581D5F60
 P 4050 2750
-F 0 "#PWR065" H 4050 2600 50  0001 C CNN
+F 0 "#PWR067" H 4050 2600 50  0001 C CNN
 F 1 "+3.3V" H 4050 2890 50  0000 C CNN
 F 2 "" H 4050 2750 50  0000 C CNN
@@
 $EndComp
 $Comp
-L GND #PWR066
+L GND #PWR068
 U 1 1 581D5F76
 P 4250 2750
-F 0 "#PWR066" H 4250 2500 50  0001 C CNN
+F 0 "#PWR068" H 4250 2500 50  0001 C CNN
 F 1 "GND" H 4250 2600 50  0000 C CNN
 F 2 "" H 4250 2750 50  0000 C CNN
@@
 	4500 4150 4500 4250
 $Comp
-L GND #PWR067
+L GND #PWR069
 U 1 1 581D6BBC
 P 4500 5100
-F 0 "#PWR067" H 4500 4850 50  0001 C CNN
+F 0 "#PWR069" H 4500 4850 50  0001 C CNN
 F 1 "GND" H 4500 4950 50  0000 C CNN
 F 2 "" H 4500 5100 50  0000 C CNN
@@
 	4050 2950 4050 2750
 $Comp
-L +3.3V #PWR068
+L +3.3V #PWR070
 U 1 1 581D6BFC
 P 4500 3400
-F 0 "#PWR068" H 4500 3250 50  0001 C CNN
+F 0 "#PWR070" H 4500 3250 50  0001 C CNN
 F 1 "+3.3V" H 4500 3540 50  0000 C CNN
 F 2 "" H 4500 3400 50  0000 C CNN
@@
 $EndComp
 Wire Wire Line
-	3900 3950 4050 3950
+	3900 3950 4200 3950
 Wire Wire Line
-	4050 3950 4200 3950
-Wire Wire Line
-	4500 3400 4500 3500
-Wire Wire Line
-	4500 3500 4500 3750
+	4500 3400 4500 3750
 $Comp
-L R R?
+L R R15
 U 1 1 582B0DCC
 P 4050 3750
-F 0 "R?" V 4130 3750 50  0000 C CNN
+F 0 "R15" V 4130 3750 50  0000 C CNN
 F 1 "10K" V 3950 3750 50  0000 C CNN
 F 2 "Resistors_SMD:R_0603_HandSoldering" V 3980 3750 50  0001 C CNN
