File: Circuit/IoTuz.kicad_pcb (KiCad board)
At the start: 2 copper layers, 150 x 95 mm, 95 parts, among them P1 ALLIGATOR_01X35, P2 BATTERY, P3 USB_5PIN_SHELL, P4 LED_1, P5 LED_2, P8 IRReceiver, Q1 S8050, Q2 S8050, Q202 FDN340P, Q203 FDN340P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

Commit message: Pushing, and shoving, and pushing.
Routing:
- net +5V: track 0.00 -> 13.4 mm
- net GND: track 2.05 -> 15.4 mm
- net /Audio/Speaker-: track 131.4 -> 129.7 mm
- net /Audio/Speaker+: track 137.4 -> 136.4 mm
Changed lines of the file:
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@@
     (thickness 1.6)
     (drawings 234)
-    (tracks 50)
+    (tracks 61)
     (zones 0)
     (modules 95)
@@
   (segment (start 64.05 119.85) (end 64.05 119) (width 0.254) (layer F.Cu) (net 1))
   (segment (start 65.75 123.05) (end 65.75 121.55) (width 0.254) (layer F.Cu) (net 1))
+  (segment (start 191 140) (end 189.668 141.332) (width 0.254) (layer F.Cu) (net 2))
+  (segment (start 189.668 141.332) (end 189.668 144) (width 0.254) (layer F.Cu) (net 2))
+  (segment (start 193.14484 140) (end 191 140) (width 0.254) (layer F.Cu) (net 2))
+  (segment (start 194.192 142.484) (end 194.192 141.04716) (width 0.254) (layer F.Cu) (net 2))
+  (segment (start 194.192 141.04716) (end 193.14484 140) (width 0.254) (layer F.Cu) (net 2))
+  (segment (start 194.192 146.242) (end 194.192 142.484) (width 0.254) (layer F.Cu) (net 2))
   (segment (start 65.25 123.05) (end 65.25 124.75) (width 0.2032) (layer F.Cu) (net 2))
   (segment (start 65.25 124.75) (end 65 125) (width 0.2032) (layer F.Cu) (net 2))
+  (segment (start 59 140) (end 60.292 141.292) (width 0.254) (layer F.Cu) (net 3))
+  (segment (start 60.292 141.292) (end 60.292 144) (width 0.254) (layer F.Cu) (net 3))
+  (segment (start 56.81516 140) (end 59 140) (width 0.254) (layer F.Cu) (net 3))
+  (segment (start 55.768 142.484) (end 55.768 141.04716) (width 0.254) (layer F.Cu) (net 3))
+  (segment (start 55.768 141.04716) (end 56.81516 140) (width 0.254) (layer F.Cu) (net 3))
+  (segment (start 55.768 146.242) (end 55.768 142.484) (width 0.254) (layer F.Cu) (net 3))
   (segment (start 66.95 124.25) (end 68.25 124.25) (width 0.254) (layer F.Cu) (net 83))
   (segment (start 68.25 124.25) (end 68.9 123.6) (width 0.254) (layer F.Cu) (net 83))
@@
   (segment (start 71.05 108) (end 71.05 108.95) (width 0.254) (layer F.Cu) (net 109))
   (segment (start 69.43 109.23) (end 65.85 109.23) (width 0.254) (layer F.Cu) (net 109))
-  (segment (start 176 135.95) (end 175.35 135.95) (width 0.254) (layer F.Cu) (net 115))
-  (segment (start 175.35 135.95) (end 173.3 138) (width 0.254) (layer F.Cu) (net 115))
-  (segment (start 173.3 138) (end 87.646592 138) (width 0.254) (layer F.Cu) (net 115))
-  (segment (start 87.646592 138) (end 78.189382 128.54279) (width 0.254) (layer F.Cu) (net 115))
-  (segment (start 78.189382 128.54279) (end 70.04279 128.54279) (width 0.254) (layer F.Cu) (net 115))
-  (segment (start 70.04279 128.54279) (end 67.75 126.25) (width 0.254) (layer F.Cu) (net 115))
-  (segment (start 67.75 126.25) (end 66.95 126.25) (width 0.254) (layer F.Cu) (net 115))
+  (segment (start 176 135.95) (end 171.05 135.95) (width 0.254) (layer F.Cu) (net 115))
+  (segment (start 82.646592 133) (end 76.55 126.903408) (width 0.254) (layer F.Cu) (net 115))
+  (segment (start 76.55 126.903408) (end 68.603408 126.903408) (width 0.254) (layer F.Cu) (net 115))
+  (segment (start 171.05 135.95) (end 168.1 133) (width 0.254) (layer F.Cu) (net 115))
+  (segment (start 168.1 133) (end 82.646592 133) (width 0.254) (layer F.Cu) (net 115))
+  (segment (start 68.603408 126.903408) (end 67.95 126.25) (width 0.254) (layer F.Cu) (net 115))
+  (segment (start 67.95 126.25) (end 66.95 126.25) (width 0.254) (layer F.Cu) (net 115))
   (segment (start 184 123.2) (end 184 125) (width 0.254) (layer F.Cu) (net 115))
   (segment (start 184 125) (end 179 130) (width 0.254) (layer F.Cu) (net 115))
@@
   (segment (start 179 130) (end 179 134) (width 0.254) (layer F.Cu) (net 115))
   (segment (start 177.05 135.95) (end 176 135.95) (width 0.254) (layer F.Cu) (net 115))
-  (segment (start 65.75 126.95) (end 65.75 127.629) (width 0.254) (layer F.Cu) (net 116))
-  (segment (start 174.139382 138.457211) (end 175.396593 137.2) (width 0.254) (layer F.Cu) (net 116))
-  (segment (start 65.75 127.629) (end 67.121001 129.000001) (width 0.254) (layer F.Cu) (net 116))
-  (segment (start 175.396593 137.2) (end 181.8 137.2) (width 0.254) (layer F.Cu) (net 116))
-  (segment (start 67.121001 129.000001) (end 78.000001 129.000001) (width 0.254) (layer F.Cu) (net 116))
-  (segment (start 78.000001 129.000001) (end 87.45721 138.457211) (width 0.254) (layer F.Cu) (net 116))
-  (segment (start 87.45721 138.457211) (end 174.139382 138.457211) (width 0.254) (layer F.Cu) (net 116))
-  (segment (start 181.8 137.2) (end 183 136) (width 0.254) (layer F.Cu) (net 116))
-  (segment (start 183 136) (end 184 135) (width 0.254) (layer F.Cu) (net 116))
+  (segment (start 184 135) (end 181.8 137.2) (width 0.254) (layer F.Cu) (net 116))
+  (segment (start 78.000001 129.000001) (end 67.121001 129.000001) (width 0.254) (layer F.Cu) (net 116))
+  (segment (start 181.8 137.2) (end 171.3 137.2) (width 0.254) (layer F.Cu) (net 116))
+  (segment (start 171.3 137.2) (end 167.55721 133.45721) (width 0.254) (layer F.Cu) (net 116))
+  (segment (start 65.75 127.629) (end 65.75 126.95) (width 0.254) (layer F.Cu) (net 116))
+  (segment (start 167.55721 133.45721) (end 82.45721 133.45721) (width 0.254) (layer F.Cu) (net 116))
+  (segment (start 82.45721 133.45721) (end 78.000001 129.000001) (width 0.254) (layer F.Cu) (net 116))
+  (segment (start 67.121001 129.000001) (end 65.75 127.629) (width 0.254) (layer F.Cu) (net 116))
   (segment (start 192 135.95) (end 184.95 135.95) (width 0.254) (layer F.Cu) (net 116))
   (segment (start 184.95 135.95) (end 184 135) (width 0.254) (layer F.Cu) (net 116))

Commit message: Nearly final positions. Looking good.
Routing:
- net GND: track 15.4 -> 11.7 mm
- net +5V: track 13.4 -> 9.64 mm
