File: Circuit/LCDTouchScreen.sch (KiCad schematic (older format))
At the start: 6 parts, among them P6 CONN_01X14, P7 CONN_01X04, Q3 FDN340P, U6 ili9341.TouchLCD.Red.NoName

Commit message: pcb footprint updates
Parts:
- P6: value CONN_01X14 -> LCD_BOM_14_NC
- P7: value CONN_01X04 -> LCD_BOM_4_NC
Changed lines of the file:
@@
 P 650 2450
 F 0 "P6" H 650 3200 50  0000 C CNN
-F 1 "CONN_01X14" V 750 2450 50  0000 C CNN
+F 1 "LCD_BOM_14_NC" V 750 2450 50  0000 C CNN
 F 2 "" H 650 2450 50  0001 C CNN
 F 3 "" H 650 2450 50  0000 C CNN
@@
 P 6250 2450
 F 0 "P7" H 6250 2700 50  0000 C CNN
-F 1 "CONN_01X04" V 6350 2450 50  0000 C CNN
+F 1 "LCD_BOM_4_NC" V 6350 2450 50  0000 C CNN
 F 2 "" H 6250 2450 50  0001 C CNN
 F 3 "" H 6250 2450 50  0000 C CNN
@@
 	3300 2000 3650 2000
 $Comp
-L +3.3V #PWR064
+L +3.3V #PWR065
 U 1 1 58242261
 P 3550 1250
-F 0 "#PWR064" H 3550 1100 50  0001 C CNN
+F 0 "#PWR065" H 3550 1100 50  0001 C CNN
 F 1 "+3.3V" H 3550 1390 50  0000 C CNN
 F 2 "" H 3550 1250 50  0000 C CNN
@@
 $EndComp
 $Comp
-L GND #PWR065
+L GND #PWR066
 U 1 1 58242289
 P 2700 1950
-F 0 "#PWR065" H 2700 1700 50  0001 C CNN
+F 0 "#PWR066" H 2700 1700 50  0001 C CNN
 F 1 "GND" H 2700 1800 50  0000 C CNN
 F 2 "" H 2700 1950 50  0000 C CNN
@@
 Connection ~ 3450 2900
 $Comp
-L +3.3V #PWR066
+L +3.3V #PWR067
 U 1 1 582B4A02
 P 2300 1700
-F 0 "#PWR066" H 2300 1550 50  0001 C CNN
+F 0 "#PWR067" H 2300 1550 50  0001 C CNN
 F 1 "+3.3V" H 2300 1840 50  0000 C CNN
 F 2 "" H 2300 1700 50  0000 C CNN

Commit message: Changes for BOM generation. Corrections to redundant BOM items.
Parts:
- U6: Non-Digikey (none) -> 1
Changed lines of the file:
@@
 F 2 "libs:lcdtouchscreen.2.8inch-red.no-name.ili9341-xpt2046" H 4300 2450 60  0001 C CNN
 F 3 "" H 4300 2450 60  0001 C CNN
+F 4 "1" H 4300 2450 60  0001 C CNN "Non-Digikey"
 	1    4300 2450
 	1    0    0    -1
